File: Data_Acquisition_Board.kicad_sch (KiCad schematic)
At the start: 0 parts

Commit message: IoT part finalization
Other:
- sheet Input&Output-ADC ports: added {MCU_ADC}; removed none
- sheet Input&Output-Command ports: added DAC1, {MCU_PWM}; removed none
- sheet MCU ports: added {MCU_ADC}, {MCU_PWM}, {MCU_Serial_COM}; removed Serial_COM
- sheet MCU IOT ports: added {MCU_Serial_COM}; removed none
- sheet Sensor ports: added {MCU_Serial_COM}; removed Serial_COM
- sheet Serial Interface ports: added {MCU_Serial_COM}; removed Serial_COM
Changed lines of the file:
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@@
 	)
 	(junction
-		(at 187.96 43.18)
+		(at 187.96 78.74)
 		(diameter 0)
 		(color 0 0 0 0)
 	)
-	(bus
-		(pts
-			(xy 184.15 43.18) (xy 187.96 43.18)
-		)
-		(stroke
-			(width 0)
-			(type default)
-		)
-	)
-	(bus
-		(pts
-			(xy 187.96 43.18) (xy 193.04 43.18)
-		)
-		(stroke
-			(width 0)
-			(type default)
-		)
-	)
-	(bus
-		(pts
-			(xy 187.96 80.01) (xy 187.96 43.18)
-		)
-		(stroke
-			(width 0)
-			(type default)
-		)
-	)
-	(bus
-		(pts
-			(xy 193.04 80.01) (xy 187.96 80.01)
+	(junction
+		(at 187.96 45.72)
+		(diameter 0)
+		(color 0 0 0 0)
+	)
+	(bus
+		(pts
+			(xy 187.96 78.74) (xy 187.96 106.68)
+		)
+		(stroke
+			(width 0)
+			(type default)
+		)
+	)
+	(bus
+		(pts
+			(xy 187.96 45.72) (xy 187.96 78.74)
+		)
+		(stroke
+			(width 0)
+			(type default)
+		)
+	)
+	(bus
+		(pts
+			(xy 105.41 121.92) (xy 105.41 106.68)
+		)
+		(stroke
+			(width 0)
+			(type default)
+		)
+	)
+	(bus
+		(pts
+			(xy 105.41 106.68) (xy 187.96 106.68)
+		)
+		(stroke
+			(width 0)
+			(type default)
+		)
+	)
+	(bus
+		(pts
+			(xy 193.04 45.72) (xy 187.96 45.72)
+		)
+		(stroke
+			(width 0)
+			(type default)
+		)
+	)
+	(bus
+		(pts
+			(xy 187.96 78.74) (xy 193.04 78.74)
+		)
+		(stroke
+			(width 0)
+			(type default)
+		)
+	)
+	(bus
+		(pts
+			(xy 97.79 86.36) (xy 120.65 86.36)
+		)
+		(stroke
+			(width 0)
+			(type default)
+		)
+	)
+	(bus
+		(pts
+			(xy 187.96 45.72) (xy 184.15 45.72)
+		)
+		(stroke
+			(width 0)
+			(type default)
+		)
+	)
+	(bus
+		(pts
+			(xy 97.79 121.92) (xy 105.41 121.92)
+		)
+		(stroke
+			(width 0)
+			(type default)
+		)
+	)
+	(bus
+		(pts
+			(xy 97.79 40.64) (xy 120.65 40.64)
 		)
 		(stroke
@@
 			)
 		)
-		(pin "Serial_COM" bidirectional
-			(at 184.15 43.18 0)
+		(pin "{MCU_ADC}" input
+			(at 120.65 40.64 180)
+			(effects
+				(font
+					(size 1.27 1.27)
+				)
+				(justify left)
+			)
+		)
+		(pin "{MCU_PWM}" output
+			(at 120.65 86.36 180)
+			(effects
+				(font
+					(size 1.27 1.27)
+				)
+				(justify left)
+			)
+		)
+		(pin "{MCU_Serial_COM}" bidirectional
+			(at 184.15 45.72 0)
 			(effects
 				(font
@@
 			)
 		)
-		(pin "Serial_COM" bidirectional
-			(at 193.04 80.01 180)
+		(pin "{MCU_Serial_COM}" bidirectional
+			(at 193.04 78.74 180)
 			(effects
 				(font
@@
 			)
 		)
-		(pin "Serial_COM" bidirectional
-			(at 193.04 43.18 180)
+		(pin "{MCU_Serial_COM}" bidirectional
+			(at 193.04 45.72 180)
 			(effects
 				(font
@@
 			)
 		)
+		(pin "{MCU_ADC}" output
+			(at 97.79 40.64 0)
+			(effects
+				(font
+					(size 1.27 1.27)
+				)
+				(justify right)
+			)
+		)
 		(instances
 			(project "Data_Acquisition_Board"
@@
 			)
 		)
+		(pin "{MCU_Serial_COM}" bidirectional
+			(at 97.79 121.92 0)
+			(effects
+				(font
+					(size 1.27 1.27)
+				)
+				(justify right)
+			)
+		)
 		(instances
 			(project "Data_Acquisition_Board"
@@
 			)
 		)
+		(pin "DAC1" input
+			(at 97.79 83.82 0)
+			(effects
+				(font
+					(size 1.27 1.27)
+				)
+				(justify right)
+			)
+		)
+		(pin "{MCU_PWM}" input
+			(at 97.79 86.36 0)
+			(effects
+				(font
+					(size 1.27 1.27)
+				)
+				(justify right)
+			)
+		)

Commit message: Release Schematic REV A-01
Other:
- sheet Input&Output-Command ports: added none; removed DAC1
- company: Blue Signal -> Nexvantis
Changed lines of the file:
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@@
 		(date "2026-07-30")
 		(rev "A-01")
-		(company "Blue Signal")
-		(comment 1 "Engineer : Franklin Jordan NZOKOU DJOKO")
-	)
-	(text_box "^ Possible ameliorations :\n	- A better GPIO estender\n	- ISO1228 for digital input between 8.5V to 36V\n	- I2C/SPI isolation : Texas instrument\n	- ACSL-7210 for UART Isolation\n	- THVD4411 For RS232 and RS485 communication"
-		(exclude_from_sim no)
-		(at 194.31 128.27 0)
-		(size 38.1 13.5716)
-		(margins 0.9525 0.9525 0.9525 0.9525)
-		(stroke
-			(width 0)
-			(type solid)
-			(color 72 72 72 1)
-		)
-		(fill
-			(type color)
-			(color 255 255 255 1)
-		)
-		(effects
-			(font
-				(face "Bahnschrift")
-				(size 1.016 1.016)
-				(color 0 0 0 1)
-			)
-			(justify left top)
-		)
-	)
-	(text_box "^ Componants choice :\n	- TCAL9539 Digital I/O\n	- LED ws2812b\n	- RS232 IC with isolation\n	- Switcher"
-		(exclude_from_sim no)
-		(at 194.31 111.76 0)
-		(size 38.1 11.43)
-		(margins 0.9525 0.9525 0.9525 0.9525)
-		(stroke
-			(width 0)
-			(type solid)
-			(color 72 72 72 1)
-		)
-		(fill
-			(type color)
-			(color 255 255 255 1)
-		)
-		(effects
-			(font
-				(face "Bahnschrift")
-				(size 1.016 1.016)
-				(color 0 0 0 1)
-			)
-			(justify left top)
-		)
+		(company "Nexvantis")
+		(comment 1 "Engineer : Jordan NZOKOU")
 	)
 	(junction
@@
 			)
 		)
-		(pin "DAC1" input
-			(at 196.85 77.47 180)
-			(effects
-				(font
-					(size 1.27 1.27)
-				)
-				(justify left)
-			)
-		)
