File: Data_Acquisition_Board.kicad_sch (KiCad schematic)
At the start: 0 parts

Commit message: [Project][Added] CI/CD environment
Other:
- removed sheet Input&Output-ADC
- removed sheet Input&Output-Command
- removed sheet MCU
- removed sheet MCU IOT
- removed sheet Power
- removed sheet Sensor
- removed sheet Serial Interface
- added sheet Block Diagram (Block Diagram.kicad_sch)
- added sheet Power - Sequencing (Power - Sequencing.kicad_sch)
- added sheet Project Architecture (Project Architecture.kicad_sch)
- added sheet Revision History (Revision History.kicad_sch)
- note added: "${BOARD_NAME}"
- note added: "${RELEASE_DATE_NUM}"
- note added: "${SHEET_NAME_10}"
- note added: "${SHEET_NAME_11}"
- note added: "${SHEET_NAME_12}"
- note added: "${SHEET_NAME_13}"
- note added: "${SHEET_NAME_14}"
- note added: "${SHEET_NAME_15}"
- note added: "${SHEET_NAME_16}"
- note added: "${SHEET_NAME_17}"
- note added: "${SHEET_NAME_18}"
- note added: "${SHEET_NAME_19}"
- note added: "${SHEET_NAME_1}"
- note added: "${SHEET_NAME_20}"
- note added: "${SHEET_NAME_21}"
- note added: "${SHEET_NAME_22}"
- note added: "${SHEET_NAME_23}"
- note added: "${SHEET_NAME_24}"
- note added: "${SHEET_NAME_25}"
- note added: "${SHEET_NAME_26}"
- note added: "${SHEET_NAME_27}"
- note added: "${SHEET_NAME_28}"
- note added: "${SHEET_NAME_29}"
- note added: "${SHEET_NAME_2}"
- note added: "${SHEET_NAME_30}"
- note added: "${SHEET_NAME_31}"
- note added: "${SHEET_NAME_32}"
- note added: "${SHEET_NAME_33}"
- note added: "${SHEET_NAME_34}"
- note added: "${SHEET_NAME_35}"
- note added: "${SHEET_NAME_36}"
- note added: "${SHEET_NAME_37}"
- note added: "${SHEET_NAME_38}"
- note added: "${SHEET_NAME_39}"
- note added: "${SHEET_NAME_3}"
- note added: "${SHEET_NAME_40}"
- note added: "${SHEET_NAME_4}"
- note added: "${SHEET_NAME_5}"
- note added: "${SHEET_NAME_6}"
- note added: "${SHEET_NAME_7}"
- note added: "${SHEET_NAME_8}"
- note added: "${SHEET_NAME_9}"
- note added: "1"
- note added: "10"
- note added: "11"
- note added: "12"
- note added: "13"
- note added: "14"
- note added: "15"
- note added: "16"
- note added: "17"
- note added: "18"
- note added: "19"
- note added: "2"
- note added: "20"
- note added: "21"
- note added: "22"
- note added: "23"
- note added: "24"
- note added: "25"
- note added: "26"
- note added: "27"
- note added: "28"
- note added: "29"
- note added: "3"
- note added: "30"
- note added: "31"
- note added: "32"
- note added: "33"
- note added: "34"
- note added: "35"
- note added: "36"
- note added: "37"
- note added: "38"
- note added: "39"
- note added: "4"
- note added: "40"
- note added: "5"
- note added: "6"
- note added: "7"
- note added: "8"
- note added: "9"
- note added: "BOTTOM VIEW"
- note added: "CHECKED - There shouldn't be any mistakes. Contact the engineer if you find any."
- note added: "Comment"
- note added: "DESIGN CONSIDERATIONS"
- note added: "DRAFT - Very early stage of schematic, ignore details."
- note added: "Date: ${RELEASE_DATE}"
- note added: "Index"
- note added: "NOTES"
- note added: "Not fitted components are marked as"
- note added: "PRELIMINARY - Close to final schematic."
- note added: "Page"
- note added: "RELEASED - A board with this schematic has been sent to production."
- note added: "Rev ${REVISION}"
- note added: "TOP VIEW"
- note added: "Variant: ${VARIANT}"
- company: Nexvantis -> ${COMPANY}
- title: Data Acquisition Board -> Sheet A
