File: Input&Output-ADC.kicad_sch (KiCad schematic)
At the start: 39 parts, among them J4 *, J5 *, J6 *, U2 G=1

Commit message: Add IOT Part
Parts:
- renumbered C13 to C?, C15 to C?, C16 to C?, C14 to C?, D4 to D?, D5 to D?, J5 to J?, J6 to J?, J4 to J?, R17 to R?, R9 to R?, R14 to R?, R12 to R?, R20 to R?, R19 to R?, R18 to R?, R13 to R?, R15 to R?, R11 to R?, R16 to R?, R10 to R?, U2 to U?
Other:
- moved on the sheet: U?E

Commit message: IoT part finalization
Connections:
- net Input10V.ADC1_IN6 renamed ADC1_IN6
- net Input10V.ADC1_IN7 renamed ADC1_IN7
- net Input3V3.ADC1_IN0 renamed ADC1_IN0
- net Input3V3.ADC1_IN1 renamed ADC1_IN1
- net Input3V3.ADC1_IN2 renamed ADC1_IN2
- net Input3V3.ADC1_IN3 renamed ADC1_IN3
- net Input5V.ADC1_IN4 renamed ADC1_IN4
- net Input5V.ADC1_IN5 renamed ADC1_IN5

Commit message: IOT part Finilization
Parts:
- removed C? (x8): 100nF, Capacitor_SMD:C_0603_1608Metric_Pad1.08x0.95mm_HandSolder, symbol Device:C_Small
- added C? (x8): 100nF, Capacitor_SMD:C_0603_1608Metric_Pad1.08x0.95mm_HandSolder, symbol Device:C_Small
- J?: Comment Analog Input 5V -> Analog Input 10V
- renumbered U2 to U?
Connections:
- net ADC1_IN0: now also C?.1
- net ADC1_IN1: now also C?.1
- net ADC1_IN2: now also C?.1
- net ADC1_IN3: now also C?.1
- net ADC1_IN4: now also C?.1
- net ADC1_IN5: now also C?.1
- net ADC1_IN6: now also C?.1
- net ADC1_IN7: now also C?.1
- net GND: now also C?.2, C?.2, C?.2, C?.2, C?.2, C?.2, C?.2, C?.2
Other:
- moved on the sheet: D?, J?, R?, U?A, U?B, U?C, U?D, U?E

Commit message: Release Schematic REV A-01
Parts:
- gave numbers to parts that had none: 35
Other:
- company: Blue Signal -> Nexvantis
