File: Input&Output-Command.kicad_sch (KiCad schematic)
At the start: 34 parts

Commit message: IoT part finalization
Parts:
- added D?: 5.5V, Package_TO_SOT_SMD:SOT-143, symbol Power_Protection:SP0503BAHT
- added J?: *, Connector_JST:JST_PH_S4B-PH-SM4-TB_1x04-1MP_P2.00mm_Horizontal, symbol Connector_Generic_MountingPin:Conn_01x04_MountingPin
- added R? (x2): 22R, Resistor_SMD:R_0603_1608Metric_Pad0.98x0.95mm_HandSolder, symbol Device:R_Small
- J?: Comment PWM1 -> GPIO_EXP_IO2
Connections:
- net +3.3V: now also D?.4 (K), J?.1 (Pin_1)
- net GND: now also D?.1 (A), J?.2 (Pin_2), J?.MP (MountPin)
- net GPIO_EXT_P16 renamed GPIO_EXP_P16
- net GPIO_EXT_P17 renamed GPIO_EXP_P17
- new net: D?.3 (K), J?.3 (Pin_3), R?.2
- new net: D?.2 (K), J?.4 (Pin_4), R?.2
- new net GPIO_EXP_P14: R?.1
- new net GPIO_EXP_P15: R?.1
Other:
- moved on the sheet: D?, J?, R?

Commit message: IOT part Finilization
Parts:
- removed D? (x4): 5.5V, Package_TO_SOT_SMD:SOT-143, symbol Power_Protection:SP0503BAHT
- added D? (x10): 3.3V, Package_TO_SOT_SMD:SOT-363_SC-70-6, symbol Power_Protection:PESD3V3L5UY
Connections:
- net +3.3V: now also D?.1 (K1), D?.1 (K1)
- net GND: now also J?.MP (MountPin), D?.2 (A), D?.2 (A)
- net at J?.4 (Pin_4), R?.2: now also D?.5 (K4) (x2)
- net at J?.4 (Pin_4), R?.2: now also D?.3 (K2) (x2)
- net at J?.3 (Pin_3), R?.2: now also D?.4 (K3) (x2)
- net at J?.3 (Pin_3), R?.2: now also D?.6 (K5) (x2)
- net LED_DIN renamed LED_PWM_DIN
Other:
- moved on the sheet: C?, D?, J?, R?

Commit message: Release Schematic REV A-01
Parts:
- gave numbers to parts that had none: 36
Connections:
- net Intput_Relay_N is gone; now on net Input_Relay_N: J13.1 (Pin_1)
- net Intput_Relay_P is gone; now on net Input_Relay_P: J13.2 (Pin_2)
- no-connect marks 0 -> 4
Other:
- company: Blue Signal -> Nexvantis
- moved on the sheet: D20A, D20B, D20C, D20D, D20E, J12, J14, R30, R31, R36, R37
