File: MCU.kicad_sch (KiCad schematic)
At the start: 39 parts, among them J1 *, J2 *, J3 *, SW1 *, U1 *, Y1 32.768kHz, Y2 16MHz

Commit message: Add IOT Part
Parts:
- renumbered C7 to C?, C8 to C?, C4 to C?, C6 to C?, C2 to C?, C11 to C?, C5 to C?, C10 to C?, C1 to C?, C9 to C?, C12 to C?, C3 to C?, D2 to D?, D3 to D?, J3 to J?, J2 to J?, R6 to R?, R7 to R?, R4 to R?, R3 to R?, R2 to R?, R8 to R?, R1 to R?, R5 to R?, Y1 to Y?, Y2 to Y?
Connections:
- net +3.3V: now also R?.2
- net GND: no longer D?.1 (K)
- net MCU_LED1: now also D?.1 (K); no longer R?.2
- net +5V_USB renamed +5V
Other:
- moved on the sheet: C?

Commit message: IoT part finalization
Parts:
- added C? (x4): 100nF, Capacitor_SMD:C_0603_1608Metric_Pad1.08x0.95mm_HandSolder, symbol Device:C_Small
- added J?: *, Connector_Molex:Molex_Micro-Fit_3.0_43045-0612_2x03_P3.00mm_Vertical, symbol Connector_Generic:Conn_02x03_Odd_Even
- added R?: 10k, Resistor_SMD:R_0603_1608Metric_Pad0.98x0.95mm_HandSolder, symbol Device:R_Small
Connections:
- net GPIO_Externter_~{INT} is gone; now on net GPIO_Expander_~{INT}: U?.1 (~{INT})
- net GPIO_Externter_~{RESET} is gone; now on net GPIO_Expander_~{RESET}: U?.3 (~{RESET})
- net +3.3V: now also C?.1, C?.1, J?.2 (Pin_2), R?.2
- net +5V: now also C?.1, C?.1, J?.4 (Pin_4)
- net DAC1: now also U1.20 (PA4)
- net GND: now also C?.2, C?.2, C?.2, C?.2, J?.6 (Pin_6)
- net I2C1_SCL: now also U1.58 (PB6)
- net I2C1_SDA: now also U1.59 (PB7)
- net I2C2_SCL: now also U1.61 (PB8)
- net I2C2_SDA: now also U1.62 (PB9)
- net IMU_SENSOR_CS: now also U1.28 (PB2); no longer U?.14 (P11)
- net LED_DIN: now also U1.57 (PB5)
- net MicroSD_CS: now also U1.54 (PD2); no longer U?.13 (P10)
- net PWM1_CH0: now also U1.41 (PA8)
- net PWM1_CH1: now also U1.50 (PA15)
- net PWM2_CH0: now also U1.55 (PB3)
- net PWM2_CH1: now also U1.56 (PB4)
- net SPI1_CS: now also U1.33 (PB12)
- net SPI1_MISO: now also U1.35 (PB14)
- net SPI1_MOSI: now also U1.36 (PB15)
- net SPI1_SCK: now also U1.34 (PB13)
- net SPI2_CS: now also U1.2 (PC13)
- net SPI2_MISO: now also U1.52 (PC11)
- net SPI2_MOSI: now also U1.53 (PC12)
- net SPI2_SCK: now also U1.51 (PC10)
- net SWCLK: now also U1.49 (PA14)
- net SWDIO: now also U1.46 (PA13)
- net Switch_DIP_1: now also U?.13 (P10); no longer U?.15 (P12)
- net Switch_DIP_2: now also U?.14 (P11); no longer U?.16 (P13)
- net Switch_DIP_3: now also U?.15 (P12); no longer U?.17 (P14)
- net Switch_DIP_4: now also U?.16 (P13); no longer U?.18 (P15)
- net UART2_MCU_RX: now also U1.38 (PC7)
- net UART2_MCU_TX: now also U1.37 (PC6)
- net ADC1_IN4: now reaches U1.14 (PA0)
- net ADC1_IN5: now reaches U1.15 (PA1)
- net ADC1_IN6: now reaches U1.16 (PA2)
- net ADC1_IN7: now reaches U1.17 (PA3)
- net MCU_SPARE1: now reaches U1.21 (PA5)
- net MCU_SPARE1: now also J?.1 (Pin_1)
- net I2C3_SDA: now reaches U1.22 (PA6)
- net I2C3_SCL: now reaches U1.23 (PA7)
- net RS_UART_MCU_TX: now reaches U1.24 (PC4)
- net RS_UART_MCU_RX: now reaches U1.25 (PC5)
- net MCU_SPARE2: now reaches U1.26 (PB0)
- net MCU_SPARE2: now also J?.3 (Pin_3)
- net MCU_SPARE3: now reaches U1.27 (PB1)
- net MCU_SPARE3: now also J?.5 (Pin_5)
- net GPIO_Expander_~{INT}: now reaches U1.39 (PC8)
- net GPIO_Expander_~{RESET}: now reaches U1.40 (PC9)
- net GPIO_Expander_~{RESET}: now also R?.1
- net Debug_UART_MCU_TX: now reaches U1.42 (PA9)
- net Debug_UART_MCU_TX: now also D?.1 (K), J?.3 (Pin_3)
- net Debug_UART_MCU_RX: now reaches U1.43 (PA10)
- net Debug_UART_MCU_RX: now also D?.2 (K), J?.4 (Pin_4)
- removed net Debug_MCU_RX: D?.2 (K), J?.4 (Pin_4), U1.29 (PB10)
- removed net Debug_MCU_TX: D?.1 (K), J?.3 (Pin_3), U1.30 (PB11)
- net GPIO_EXT_P16 renamed GPIO_EXP_P16
- net GPIO_EXT_P17 renamed GPIO_EXP_P17
- net I2C1.SCL renamed I2C2.SCL
- net I2C1.SDA renamed I2C2.SDA
- net Input3V3.ADC1_IN0 renamed ADC1_IN0
- net Input3V3.ADC1_IN1 renamed ADC1_IN1
- net Input3V3.ADC1_IN2 renamed ADC1_IN2
- net Input3V3.ADC1_IN3 renamed ADC1_IN3
- new net GPIO_EXP_P14: U?.17 (P14)
- new net GPIO_EXP_P15: U?.18 (P15)
- new net IOT_UART_MCU_RX: U1.30 (PB11)
- new net IOT_UART_MCU_TX: U1.29 (PB10)
Other:
- note added: "GPIO Expander"
- note added: "MCU SPARE CONNECTOR"
- note removed: "GPIO Extender"
- moved on the sheet: BT?, C?, D1A, D1B, D1C, D1D, D1E, D?, F2, J1, J?, R?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

Commit message: IOT part Finilization
Parts:
- added R?: 10k, Resistor_SMD:R_0603_1608Metric_Pad0.98x0.95mm_HandSolder, symbol Device:R_Small
Connections:
- net Debug_UART_MCU_RX: now also D?.1 (K); no longer D?.2 (K)
- net Debug_UART_MCU_TX: now also D?.2 (K); no longer D?.1 (K)
- net GND: now also R?.2
- net MCU_BOOT0: now reaches U1.60 (PF3)
- net MCU_BOOT0: now also R?.1
- net LED_DIN renamed LED_PWM_DIN
Other:
- moved on the sheet: C?, D?

Commit message: Add power part : LDO and SMPS regulators
Parts:
- R? (x2): footprint Resistor_SMD:R_0603_1608Metric_Pad0.98x0.95mm_HandSolder -> Resistor_SMD:R_0805_2012Metric_Pad1.20x1.40mm_HandSolder; PackageReference 0603 -> 0805
- renumbered F2 to F?
Other:
- moved on the sheet: R?
Changed lines of the file:
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@@
 	)
 	(junction
-		(at 82.55 185.42)
+		(at 166.37 81.28)
 		(diameter 0)
 		(color 0 0 0 0)
 	)
 	(junction
-		(at 166.37 81.28)
+		(at 82.55 185.42)
 		(diameter 0)
 		(color 0 0 0 0)
@@
 	)
 	(junction
-		(at 209.55 111.76)
+		(at 152.4 81.28)
 		(diameter 0)
 		(color 0 0 0 0)
 	)
 	(junction
-		(at 81.28 156.21)
+		(at 209.55 111.76)
 		(diameter 0)
 		(color 0 0 0 0)
 	)
 	(junction
-		(at 152.4 29.21)
+		(at 81.28 156.21)
 		(diameter 0)
 		(color 0 0 0 0)
 	)
 	(junction
-		(at 31.75 176.53)
+		(at 152.4 29.21)
 		(diameter 0)
 		(color 0 0 0 0)
 	)
 	(junction
-		(at 152.4 81.28)
+		(at 31.75 176.53)
 		(diameter 0)
 		(color 0 0 0 0)
@@
 	(wire
 		(pts
-			(xy 166.37 82.55) (xy 166.37 81.28)
+			(xy 166.37 83.82) (xy 166.37 81.28)
 		)
 		(stroke
@@
 	(wire
 		(pts
-			(xy 166.37 81.28) (xy 162.56 81.28)
+			(xy 166.37 81.28) (xy 163.83 81.28)
 		)
 		(stroke
@@
 	(wire
 		(pts
-			(xy 166.37 87.63) (xy 166.37 88.9)
+			(xy 166.37 88.9) (xy 166.37 90.17)
 		)
 		(stroke
@@
 	(wire
 		(pts
-			(xy 152.4 81.28) (xy 157.48 81.28)
+			(xy 152.4 81.28) (xy 158.75 81.28)
 		)
 		(stroke
@@
 	(symbol
 		(lib_id "power:GND")
-		(at 166.37 88.9 0)
+		(at 166.37 90.17 0)
 		(unit 1)
 		(body_style 1)
@@
 		(dnp no)
 		(property "Reference" "#PWR02"
-			(at 166.37 95.25 0)
+			(at 166.37 96.52 0)
 			(hide yes)
 			(show_name no)
@@
 		)
 		(property "Value" "GND"
-			(at 166.37 92.71 0)
+			(at 166.37 93.98 0)
 			(show_name no)
 			(do_not_autoplace no)
@@
 		)
 		(property "Footprint" ""
-			(at 166.37 88.9 0)
+			(at 166.37 90.17 0)
 			(hide yes)
 			(show_name no)
@@
 		)
 		(property "Datasheet" ""
-			(at 166.37 88.9 0)
+			(at 166.37 90.17 0)
 			(hide yes)
 			(show_name no)
@@
 		)
 		(property "Description" "Power symbol creates a global label with name \"GND\" , ground"
-			(at 166.37 88.9 0)
+			(at 166.37 90.17 0)
 			(hide yes)
 			(show_name no)
@@
 	(symbol
 		(lib_id "Device:R_Small")
-		(at 166.37 85.09 0)
+		(at 166.37 86.36 0)
 		(unit 1)
 		(body_style 1)
@@
 		(dnp no)
 		(property "Reference" "R?"
-			(at 164.338 85.09 0)
+			(at 164.338 86.36 0)
 			(show_name no)
 			(do_not_autoplace no)
@@
 		)
 		(property "Value" "9.1k"
-			(at 169.418 85.09 0)
+			(at 169.418 86.36 0)
 			(show_name no)
 			(do_not_autoplace no)
@@
 			)
 		)
-		(property "Footprint" "Resistor_SMD:R_0603_1608Metric_Pad0.98x0.95mm_HandSolder"
-			(at 166.37 85.09 0)
+		(property "Footprint" "Resistor_SMD:R_0805_2012Metric_Pad1.20x1.40mm_HandSolder"
+			(at 166.37 86.36 0)
 			(hide yes)
 			(show_name no)
@@
 		)
 		(property "Datasheet" ""
-			(at 166.37 85.09 0)
+			(at 166.37 86.36 0)
 			(hide yes)
 			(show_name no)
@@
 		)
 		(property "Description" "Chip Resistor, 1%  100ppm/°C  50V"
-			(at 166.37 85.09 0)
+			(at 166.37 86.36 0)
 			(hide yes)
 			(show_name no)
@@
 		)
 		(property "PartNumber" "*"
-			(at 166.37 85.09 90)
+			(at 166.37 86.36 90)
 			(hide yes)
 			(show_name no)
@@
 			)
 		)
-		(property "PackageReference" "0603"
-			(at 166.37 85.09 90)
+		(property "PackageReference" "0805"
+			(at 166.37 86.36 90)
 			(hide yes)
 			(show_name no)
@@
 		)
 		(property "Manufacturer" "*"
-			(at 166.37 85.09 90)
+			(at 166.37 86.36 90)
 			(hide yes)
 			(show_name no)
@@
 		)
 		(property "Comment" "Resistor"
-			(at 166.37 85.09 90)
+			(at 166.37 86.36 90)
 			(hide yes)
 			(show_name no)
@@
 		(dnp no)
 		(property "Reference" "R?"
-			(at 130.302 99.314 90)
+			(at 129.54 99.314 90)
 			(show_name no)
 			(do_not_autoplace no)
@@
 		(dnp no)
 		(property "Reference" "R?"
-			(at 130.302 101.854 90)
+			(at 129.54 101.854 90)
 			(show_name no)
 			(do_not_autoplace no)
@@
 		(in_pos_files yes)
 		(dnp no)
-		(property "Reference" "F2"
+		(property "Reference" "F?"
 			(at 135.89 79.502 0)
 			(show_name no)
@@
 			(project "Data_Acquisition_Board"
 				(path "/0a00d473-e3b0-43fe-b305-746583278f51/010e493e-f38b-4bcf-bb40-d616c0d1b790"
-					(reference "F2")
+					(reference "F?")
 					(unit 1)
 				)
@@
 	(symbol
 		(lib_id "Device:R_Small")
-		(at 160.02 81.28 270)
+		(at 161.29 81.28 270)
 		(unit 1)
 		(body_style 1)
@@
 		(dnp no)
 		(property "Reference" "R?"
-			(at 160.02 77.47 90)
+			(at 161.29 77.47 90)
 			(show_name no)
 			(do_not_autoplace no)
@@
 		)
 		(property "Value" "4.7k"
-			(at 160.02 79.502 90)
+			(at 161.29 79.502 90)
 			(show_name no)
 			(do_not_autoplace no)
@@
 			)
 		)
-		(property "Footprint" "Resistor_SMD:R_0603_1608Metric_Pad0.98x0.95mm_HandSolder"
-			(at 160.02 81.28 0)
+		(property "Footprint" "Resistor_SMD:R_0805_2012Metric_Pad1.20x1.40mm_HandSolder"
+			(at 161.29 81.28 0)
 			(hide yes)
 			(show_name no)
@@
 		)
 		(property "Datasheet" ""
-			(at 160.02 81.28 0)
+			(at 161.29 81.28 0)
 			(hide yes)
 			(show_name no)
@@
 		)
 		(property "Description" "Chip Resistor, 1%  100ppm/°C  50V"
-			(at 160.02 81.28 0)
+			(at 161.29 81.28 0)
 			(hide yes)
 			(show_name no)
@@
 		)
 		(property "PartNumber" "*"
-			(at 160.02 81.28 90)
+			(at 161.29 81.28 90)
 			(hide yes)
 			(show_name no)
@@
 			)
 		)
-		(property "PackageReference" "0603"
-			(at 160.02 81.28 90)
+		(property "PackageReference" "0805"
+			(at 161.29 81.28 90)
 			(hide yes)
 			(show_name no)
@@
 		)
 		(property "Manufacturer" "*"
-			(at 160.02 81.28 90)
+			(at 161.29 81.28 90)
 			(hide yes)
 			(show_name no)
@@
 		)
 		(property "Comment" "Resistor"
-			(at 160.02 81.28 90)
+			(at 161.29 81.28 90)
 			(hide yes)
 			(show_name no)

Commit message: Release Schematic REV A-01
Parts:
- removed U?: TCAL9539, Package_SO:TSSOP-24_4.4x7.8mm_P0.65mm, symbol P_Interface:TCA9535PWR
- added U2: TCAL9539, Package_SO:TSSOP-24_4.4x7.8mm_P0.65mm, symbol P_Interface:TCA9535PWR
- gave numbers to parts that had none: 41
Connections:
- net +3.3V: now also U2.24 (VCC)
- net CD_RELAY1: now also U2.10 (P06)
- net CD_RELAY2: now also U2.11 (P07)
- net GND: now also U2.12 (GND), U2.2 (A1), U2.21 (A0)
- net GPIO_EXP_P14: now also U2.17 (P14)
- net GPIO_EXP_P15: now also U2.18 (P15)
- net GPIO_EXP_P16: now also U2.19 (P16)
- net GPIO_EXP_P17: now also U2.20 (P17)
- net GPIO_Expander_~{INT}: now also U2.1 (~{INT})
- net GPIO_Expander_~{RESET}: now also U2.3 (~{RESET})
- net I2C2_SCL: now also U2.22 (SCL)
- net I2C2_SDA: now also U2.23 (SDA)
- net IMU_SENSOR_INT1: now also U2.4 (P00)
- net IMU_SENSOR_INT2: now also U2.5 (P01)
- net Light_SENSOR_INT: now also U2.6 (P02)
- net MCU_LED1: now also U1.21 (PA5)
- net MCU_SPARE1: now also U1.26 (PB0); no longer U1.21 (PA5)
- net MCU_SPARE2: now also U1.27 (PB1); no longer U1.26 (PB0)
- net MicroSD_Detection: now also U2.7 (P03)
- net RS485_DE: now also U2.9 (P05)
- net RS485_~{RE}: now also U2.8 (P04)
- net Switch_DIP_1: now also U2.13 (P10)
- net Switch_DIP_2: now also U2.14 (P11)
- net Switch_DIP_3: now also U2.15 (P12)
- net Switch_DIP_4: now also U2.16 (P13)
- net MCU_SPARE3: no longer names the net of J4.5 (Pin_5)
- net MCU_SPARE3: no longer U1.27 (PB1)
- no-connect marks 3 -> 4
Other:
- note added: "Programming"
- note removed: "Programmation"
- company: Blue Signal -> Nexvantis
