File: Power.kicad_sch (KiCad schematic)
At the start: 0 parts

Commit message: Add power part : LDO and SMPS regulators
Parts:
- added C? (x2): 100uF, Capacitor_SMD:C_0805_2012Metric_Pad1.18x1.45mm_HandSolder, symbol Device:C_Small
- added C? (x3): 22uF, Capacitor_SMD:C_0805_2012Metric_Pad1.18x1.45mm_HandSolder, symbol Device:C_Small
- added C?: 10uF, Capacitor_SMD:CP_Elec_5x5.3, symbol Device:C_Polarized_Small
- added C?: 100uF, Capacitor_Tantalum_SMD:CP_EIA-7343-15_Kemet-W_HandSolder, symbol Device:C_Polarized_Small
- added C? (x2): 10uF, Capacitor_SMD:C_0805_2012Metric_Pad1.18x1.45mm_HandSolder, symbol Device:C_Small
- added L?: 3.3uF, PCM_SparkFun-Coil:Inductor_4.7x4.7mm, symbol PCM_SparkFun-Coil:10uH_5x5mm_1.0A
- added R?: 54.9k, Resistor_SMD:R_0805_2012Metric_Pad1.20x1.40mm_HandSolder, symbol Device:R_Small
- added R? (x2): 10k, Resistor_SMD:R_0805_2012Metric_Pad1.20x1.40mm_HandSolder, symbol Device:R_Small
- added U?: 3V3, Package_TO_SOT_SMD:TO-263-3_TabPin2, symbol Regulator_Linear:LM1085-3.3
- added U?: 5V, Package_TO_SOT_SMD:SOT-23-6, symbol Regulator_Switching:TPS563200
Connections:
- new net: C?.1, L?.1, U?.2 (SW)
- new net: C?.2, U?.6 (VBST)
- new net: R?.1, R?.2, U?.4 (VFB)
- new net: R?.1, U?.5 (EN)
- new net +3.3V: C?.1, U?.2 (VO)
- new net +5V: C?.1, C?.1, C?.1, C?.1, L?.2, R?.2, U?.3 (VI)
- new net GND: C?.2, C?.2, C?.2, C?.2, C?.2, C?.2, C?.2, C?.2, R?.1, U?.1 (GND), U?.1 (GND)
- new net Vout_Protections: C?.1, C?.1, C?.1, R?.2, U?.3 (VIN)
Other:
- note added: "3V3 LDO Regulator"
- note added: "5V SMPS Regulator"
- note added: "Vin = 7V to 17V (7366mW minimum)"

Commit message: Release Schematic REV A-01
Parts:
- added D30: 13V, Diode_SMD:D_SOD-123F, symbol Diode:BZT52Bxx
- added D31: 22V, Diode_SMD:D_0603_1608Metric_Pad1.05x0.95mm_HandSolder, symbol Device:D_TVS
- added D32: 18V, Diode_SMD:D_SOD-123F, symbol Diode:BZT52Bxx
- added D33: 2A, Diode_SMD:D_SMB, symbol Device:D_Small
- added F3: 2A, Fuse:Fuse_2920_7451Metric_Pad2.10x5.45mm_HandSolder, symbol Device:Fuse_Small
- added J35, J37: *, Connector_Wire:SolderWirePad_1x01_SMD_4x8mm, symbol Connector_Generic:Conn_01x01
- added J36: *, Connector_BarrelJack:BarrelJack_Horizontal, symbol Connector:Barrel_Jack_MountingPin
- added Q3: *, Package_TO_SOT_SMD:TO-263-3_TabPin2, symbol PCM_SparkFun-DiscreteSemi:Q_PMOS_GDS
- added R80: 100k, Resistor_SMD:R_0805_2012Metric_Pad1.20x1.40mm_HandSolder, symbol Device:R_Small
- added R81: 10k, Resistor_SMD:R_0805_2012Metric_Pad1.20x1.40mm_HandSolder, symbol Device:R_Small
- gave numbers to parts that had none: 15
Connections:
- net +5V: now also D33.1 (K)
- net GND: now also D31.1 (A1), D32.2 (A), D33.2 (A), J36.2, J36.MP (MountPin), J37.1 (Pin_1), R81.1
- net Vout_Protections: now also D30.1 (K), Q3.3 (S), R80.2
- new net: D30.2 (A), Q3.1 (G), R80.1, R81.2
- new net: F3.1, J35.1 (Pin_1), J36.1
- new net: D31.2 (A2), D32.1 (K), F3.2, Q3.2 (D)
Other:
- note added: "Protections"
- company: Blue Signal -> Nexvantis
- moved on the sheet: C58, C59, C60, C61, C62, C63, C64, C65, C66, L1, R82, R83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
