File: Data-Acquisition-Board.kicad_sch (KiCad schematic)
At the start: 0 parts

Commit message: [Project][Added] CI/CD environment
Other:
- title: Sheet A -> (none)
Changed lines of the file:
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@@
 (kicad_sch
-	(version 20260306)
+	(version 20250114)
 	(generator "eeschema")
-	(generator_version "10.0")
+	(generator_version "9.0")
 	(paper "A3")
 	(title_block
-		(title "Sheet A")
 		(date "2025-01-12")
 		(rev "${REVISION}")
@@
 		)
 		(fill
-			(color 0 0 0 0)
+			(color 0 0 0 0.0000)
 		)
 		(property "Sheetname" "Power - Sequencing"
 			(at 340.36 312.6609 0)
-			(show_name no)
-			(do_not_autoplace no)
 			(effects
 				(font
@@
 		(property "Sheetfile" "Power - Sequencing.kicad_sch"
 			(at 341.63 314.96 0)
-			(show_name no)
-			(do_not_autoplace no)
 			(effects
 				(font
@@
 		)
 		(instances
-			(project "Data_Acquisition_Board"
+			(project "Data-Acquisition-Board"
 				(path "/f9e05184-c88b-4a88-ae9c-ab2bdb32be7c"
 					(page "11")
@@
 		)
 		(fill
-			(color 0 0 0 0)
+			(color 0 0 0 0.0000)
 		)
 		(property "Sheetname" "Revision History"
 			(at 340.36 300.99 0)
-			(show_name no)
-			(do_not_autoplace no)
 			(effects
 				(font
@@
 		(property "Sheetfile" "Revision History.kicad_sch"
 			(at 340.995 303.53 0)
-			(show_name no)
-			(do_not_autoplace no)
 			(effects
 				(font
@@
 		)
 		(instances
-			(project "Data_Acquisition_Board"
+			(project "Data-Acquisition-Board"
 				(path "/f9e05184-c88b-4a88-ae9c-ab2bdb32be7c"
 					(page "12")
@@
 		)
 		(fill
-			(color 0 0 0 0)
+			(color 0 0 0 0.0000)
 		)
 		(property "Sheetname" "Block Diagram"
 			(at 299.72 301.2309 0)
-			(show_name no)
-			(do_not_autoplace no)
 			(effects
 				(font
@@
 		(property "Sheetfile" "Block Diagram.kicad_sch"
 			(at 300.99 303.53 0)
-			(show_name no)
-			(do_not_autoplace no)
 			(effects
 				(font
@@
 		)
 		(instances
-			(project "Data_Acquisition_Board"
+			(project "Data-Acquisition-Board"
 				(path "/f9e05184-c88b-4a88-ae9c-ab2bdb32be7c"
 					(page "2")
@@
 		)
 		(fill
-			(color 0 0 0 0)
+			(color 0 0 0 0.0000)
 		)
 		(property "Sheetname" "Project Architecture"
 			(at 299.72 312.6609 0)
-			(show_name no)
-			(do_not_autoplace no)
 			(effects
 				(font
@@
 		(property "Sheetfile" "Project Architecture.kicad_sch"
 			(at 300.99 314.96 0)
-			(show_name no)
-			(do_not_autoplace no)
 			(effects
 				(font
@@
 		)
 		(instances
-			(project "Data_Acquisition_Board"
+			(project "Data-Acquisition-Board"
 				(path "/f9e05184-c88b-4a88-ae9c-ab2bdb32be7c"
 					(page "3")
