File: In&Out - ADC.kicad_sch (KiCad schematic)
At the start: 47 parts

Commit message: [Schematic][Modify] Annotation of all  the components
Parts:
- gave numbers to parts that had none: 35

Commit message: [Schematic][Modify] Annotation of all  the components
Parts:
- renumbered C32 to C30, C36 to C31, C33 to C32, C37 to C33, C30 to C35, C31 to C36, C35 to C37, D12 to D11, D15 to D12, D16 to D13, D18 to D14, D20 to D15, D14 to D16, D19 to D17, D11 to D18, D13 to D19, D17 to D20, J13 to J11, J11 to J12, J12 to J13, R33 to R28, R34 to R29, R35 to R30, R36 to R31, R30 to R32, R31 to R33, R37 to R34, R39 to R35, R28 to R36, R29 to R37, R32 to R38, R38 to R39, U6 to U5, U5 to U6
